File: STM32L431RCT6_prototype_board.kicad_sch (KiCad schematic)
At the start: 30 parts, among them J10 SWD, J2 Conn_02x20_Counter_Clockwise, U1 STM32L431CCTx, U3 SY8089, Y1 8MHz

Commit message: add gerber.
Parts:
- added F1: Fuse, Fuse:Fuse_1812_4532Metric, symbol Device:Fuse
Connections:
- net RCC_MCO is gone; now on net PA8: U1.29 (PA8)
- net +3V3: now also J2.37 (Pin_37)
- net +5.0V: now also F1.2; no longer J2.40 (Pin_40)
- net BOOT0: now also J2.22 (Pin_22)
- net NRST: now also J2.38 (Pin_38)
- net PA0: now reaches U1.10 (PA0)
- net PA0: now also J2.3 (Pin_3)
- net PA1: now reaches U1.11 (PA1)
- net PA1: now also J2.4 (Pin_4)
- net PA2: now reaches U1.12 (PA2)
- net PA2: now also J2.5 (Pin_5)
- net PA3: now reaches U1.13 (PA3)
- net PA3: now also J2.6 (Pin_6)
- net PA4: now reaches U1.14 (PA4)
- net PA4: now also J2.7 (Pin_7)
- net PA5: now reaches U1.15 (PA5)
- net PA5: now also J2.8 (Pin_8)
- net PA6: now reaches U1.16 (PA6)
- net PA6: now also J2.9 (Pin_9)
- net PA7: now reaches U1.17 (PA7)
- net PA7: now also J2.10 (Pin_10)
- net PB0: now reaches U1.18 (PB0)
- net PB0: now also J2.11 (Pin_11)
- net PB1: now reaches U1.19 (PB1)
- net PB1: now also J2.12 (Pin_12)
- net PB2: now reaches U1.20 (PB2)
- net PB2: now also J2.13 (Pin_13)
- net PB10: now reaches U1.21 (PB10)
- net PB10: now also J2.14 (Pin_14)
- net PB11: now reaches U1.22 (PB11)
- net PB11: now also J2.15 (Pin_15)
- net PB12: now reaches U1.25 (PB12)
- net PB12: now also J2.16 (Pin_16)
- net PB13: now reaches U1.26 (PB13)
- net PB13: now also J2.17 (Pin_17)
- net PB14: now reaches U1.27 (PB14)
- net PB14: now also J2.18 (Pin_18)
- net PB15: now reaches U1.28 (PB15)
- net PB15: now also J2.19 (Pin_19)
- net PC14: now reaches U1.3 (PC14)
- net PC14: now also J2.35 (Pin_35)
- net PA9: now reaches U1.30 (PA9)
- net PA9: now also J2.24 (Pin_24)
- net PA10: now reaches U1.31 (PA10)
- net PA10: now also J2.25 (Pin_25)
- net PA11: now reaches U1.32 (PA11)
- net PA11: now also J2.26 (Pin_26)
- net PA12: now reaches U1.33 (PA12)
- net PA12: now also J2.27 (Pin_27)
- net PA15: now reaches U1.38 (PA15)
- net PA15: now also J2.28 (Pin_28)
- net PC15: now reaches U1.4 (PC15)
- net PC15: now also J2.36 (Pin_36)
- net PB4: now reaches U1.40 (PB4)
- net PB4: now also J2.29 (Pin_29)
- net PB5: now reaches U1.41 (PB5)
- net PB5: now also J2.30 (Pin_30)
- net PB6: now reaches U1.42 (PB6)
- net PB6: now also J2.31 (Pin_31)
- net PB7: now reaches U1.43 (PB7)
- net PB7: now also J2.32 (Pin_32)
- net PB8: now reaches U1.45 (PB8)
- net PB8: now also J2.33 (Pin_33)
- net PB9: now reaches U1.46 (PB9)
- net PB9: now also J2.34 (Pin_34)
- net PA8: now reaches J2.23 (Pin_23)
- new net +5V: F1.1, J2.40 (Pin_40)
- no-connect marks 6 -> 0
Other:
- moved on the sheet: J2
