File: STM32L431RCT6_prototype_board.kicad_pcb (KiCad board)
At the start: 4 copper layers, 51.6 x 20.2 mm, 31 parts, among them J1 SWD, J2 Conn_02x20_Counter_Clockwise, U1 STM32L431CCTx, U2 SY8089, Y1 8MHz

Commit message: add gerber.
Routing:
- net NRST: track 52.7 -> 49.6 mm, vias 4 -> 5
- net GND: track 38.2 -> 39.9 mm, vias 16 -> 14
- net +3V3: track 20.9 -> 21.6 mm

Commit message: Update STM32L431RCT6_prototype_board.kicad_pcb
Other:
- board text added: "STM32L431CCT6"
Changed lines of the file:
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@@
   (gr_arc locked (start 157.3 53.25) (mid 157.592893 52.542893) (end 158.3 52.25)
     (stroke (width 0.1) (type default)) (layer "Edge.Cuts"))
+  (gr_poly
+    (pts
+      (xy 161 50)
+      (xy 161.48 51.6)
+      (xy 161.96 50)
+    )
+    (stroke (width 0.15) (type solid)) (fill solid) (layer "User.4"))
+  (gr_poly
+    (pts
+      (xy 166 50)
+      (xy 166.48 51.6)
+      (xy 166.96 50)
+    )
+    (stroke (width 0.15) (type solid)) (fill solid) (layer "User.4"))
+  (gr_poly
+    (pts
+      (xy 212 56.6)
+      (xy 210.4 57.08)
+      (xy 212 57.56)
+    )
+    (stroke (width 0.15) (type solid)) (fill solid) (layer "User.4"))
+  (gr_poly
+    (pts
+      (xy 163.52 50)
+      (xy 164 51.6)
+      (xy 164.48 50)
+    )
+    (stroke (width 0.15) (type solid)) (fill solid) (layer "User.4"))
   (gr_text "C15" (at 169.16 53.6) (layer "F.SilkS")
     (effects (font (size 0.9 0.7) (thickness 0.15)) (justify bottom))
@@
     (effects (font (size 0.9 0.7) (thickness 0.15)) (justify bottom))
   )
+  (gr_text "STM32L431CCT6" (at 216.8 57.6) (layer "F.SilkS")
+    (effects (font (size 0.9 0.7) (thickness 0.15)) (justify bottom))
+  )
   (gr_text "A4" (at 174.24 72.15) (layer "F.SilkS")
     (effects (font (size 0.9 0.7) (thickness 0.15)) (justify bottom))
@@
   )
   (gr_text "B14" (at 202.18 72.15) (layer "F.SilkS")
+    (effects (font (size 0.9 0.7) (thickness 0.15)) (justify bottom))
+  )
+  (gr_text "3V3" (at 166.6 49.6) (layer "F.SilkS")
     (effects (font (size 0.9 0.7) (thickness 0.15)) (justify bottom))
   )
@@
   )
   (gr_text "A11" (at 194.56 53.6) (layer "F.SilkS")
+    (effects (font (size 0.9 0.7) (thickness 0.15)) (justify bottom))
+  )
+  (gr_text "NC" (at 161.6 49.6) (layer "F.SilkS")
     (effects (font (size 0.9 0.7) (thickness 0.15)) (justify bottom))
   )
@@
     (effects (font (size 0.9 0.7) (thickness 0.15)) (justify bottom))
   )
+  (gr_text "RST" (at 164 49.6) (layer "F.SilkS")
+    (effects (font (size 0.9 0.7) (thickness 0.15)) (justify bottom))
+  )
